File: STM32G4_USB_PD.kicad_pcb (KiCad board)
At the start: 2 copper layers, 34 x 24 mm, 22 parts, among them J1 USB4105-GF-A, J2 8.06.16_J-LINK_6-PIN_NEEDLE_A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, J3 Conn_01x04, J4 Conn_01x02, Q1 2N7002K, U1 STM32G431C8T6, U2 AP2205-W5-7

Commit message: add usb-C, USB Device and PWM firmware
Connections:
- U1 pad 25: USART2_RX -> USART3_RX
Routing:
- net USART2_RX: track 25.3 -> 22.6 mm
Changed lines of the file:
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@@
   (net 43 "Net-(D2-Pad1)")
   (net 44 "Net-(D1-Pad2)")
+  (net 45 "USART3_RX")
   (footprint "J-LINK_6-PIN_NEEDLE_ADAPTER:J-LINK_6-PIN_NEEDLE_ADAPTER" (layer "F.Cu")
     (at 111 86.5 180)
@@
       (net 5 "+3.3V") (pinfunction "VDD") (pintype "power_in"))
     (pad "25" smd rect (at 4.249999 2.75 180) (size 1.1938 0.3048) (layers "F.Cu" "F.Paste" "F.Mask")
-      (net 13 "USART2_RX") (pinfunction "PB11") (pintype "bidirectional"))
+      (net 45 "USART3_RX") (pinfunction "PB11") (pintype "bidirectional"))
     (pad "26" smd rect (at 4.249999 2.250001 180) (size 1.1938 0.3048) (layers "F.Cu" "F.Paste" "F.Mask")
       (net 30 "unconnected-(U1-Pad26)") (pinfunction "PB12") (pintype "bidirectional+no_connect"))
@@
   (segment (start 108.9543 74.5406) (end 109.7607 73.7342) (width 0.2) (layer "F.Cu") (net 13))
   (segment (start 109.7607 73.7342) (end 112.7738 73.7342) (width 0.2) (layer "F.Cu") (net 13))
-  (segment (start 104.2738 73.2342) (end 105.171 73.2342) (width 0.2) (layer "F.Cu") (net 13))
   (segment (start 106.2911 74.5406) (end 108.9543 74.5406) (width 0.2) (layer "F.Cu") (net 13))
-  (segment (start 105.171 73.4205) (end 106.2911 74.5406) (width 0.2) (layer "F.Cu") (net 13))
-  (segment (start 105.171 73.2342) (end 105.171 73.4205) (width 0.2) (layer "F.Cu") (net 13))
   (via (at 106.2911 74.5406) (size 0.5) (drill 0.3) (layers "F.Cu" "B.Cu") (net 13))
   (segment (start 100.5 80.3317) (end 106.2911 74.5406) (width 0.2) (layer "B.Cu") (net 13))
